File: Lab5/lab5.sch (EAGLE design)
At the start: 53 parts, among them J1 ISP, U1 ATMEGA128RFA1

Commit message: Revamped the lab 5 schematic
Cleaned up the schematic a bunch and condensed the libraries into 1
called lab5_comps.lbr
Parts:
- removed U$3, U$4, U$5, U$6: FET, copter_components:FET
- added C18: 1uF, lab5_comps:C-USC0805
- added Q1, Q2, Q3, Q4: SI2302CDS, lab5_comps:SI2302CDS
- B1: device Lab5:BALUN0805 -> lab5_comps:BALUN0805
- C1, C10, C11, C13, C14, C15, C2, C3, C4, C5, C6, C7, C8, C9: device Lab5:C-USC0805 -> lab5_comps:C-USC0805
- C12: value 1uF -> 0.01uF; device Lab5:C-USC0805 -> lab5_comps:C-USC0805
- C16, C17: value (none) -> JUMP; device Lab5:C-USC0805 -> lab5_comps:C-USC0805
- D1, D2, D3, D4: value DIODE -> BAS16WS; device copter_components:DIODE -> lab5_comps:BAS16WS
- J1: device Lab5:AVR_SPI_PRG_6NS -> lab5_comps:AVR_SPI_PRG_6NS
- JP1: device Lab5:FTDI_BASICPTH -> lab5_comps:FTDI_BASICPTH
- JP2: value (none) -> Battery; device Lab5:M02PTH -> lab5_comps:M02PTH
- JP3: value FTDI -> Serial Debugger; device Lab5:FTDI_BASICPTH -> lab5_comps:FTDI_BASICPTH
- LED1, LED2, LED3: device Lab5:LEDCHIP-LED0805 -> lab5_comps:LEDCHIP-LED0805
- MOT1, MOT2, MOT3, MOT4: value (none) -> 20mm; device Lab5:M02PTH -> lab5_comps:M02PTH
- R1, R10, R2, R3, R4, R9: device Lab5:R-US_R0805 -> lab5_comps:R-US_R0805
- R5, R6, R7, R8: value (none) -> 10k; device Lab5:R-US_R0805 -> lab5_comps:R-US_R0805
- S1: value (none) -> On/Off; device Lab5:SWITCH-SPDTPTH -> lab5_comps:SWITCH-SPDTPTH
- U$1: device Lab5:ANTENNA2SMD5 -> lab5_comps:ANTENNA2SMD5
- U$2: device Lab5:LP3985IM5-3.0 -> lab5_comps:LP3985IM5-3.0
- U$7: device lab4_comps:LSM9DS0 -> lab5_comps:LSM9DS0
- U1: device Lab5:ATMEGA128RFA1 -> lab5_comps:ATMEGA128RFA1
- Y1: value (none) -> 16MHz; device Lab5:CRYSTAL5X3 -> lab5_comps:CRYSTAL5X3
Connections:
- net N$13 renamed RFN
- net N$14 renamed RFP
- removed net SCH: J1.3
- net 3V: now also C18.1, D1.P$1, D2.P$1, D3.P$1, D4.P$1, U$7.VDD@1, U$7.VDD@2, U$7.VDD@3, U$7.VDD_IO; no longer D1.P$NEG, D2.P$NEG, D3.P$NEG, D4.P$NEG, U$7.P$15, U$7.P$16, U$7.P$17, U$7.P$18
- net GND: now also C18.2, Q1.P$2, Q2.P$2, Q3.P$2, Q4.P$2, U$7.GND@1, U$7.GND@2, U$7.GND@3, U$7.GND@4, U$7.GND@5, U$7.SA0_G, U$7.SA0_XM; no longer U$3.P$2, U$4.P$2, U$5.P$2, U$6.P$2, U$7.P$2, U$7.P$22, U$7.P$23, U$7.P$3, U$7.P$4, U$7.P$5, U$7.P$6
- net N$18: now also D1.P$2, Q1.P$3; no longer D1.P$POS, U$3.P$3
- net N$20: now also D2.P$2, Q2.P$3; no longer D2.P$POS, U$4.P$3
- net N$22: now also D3.P$2, Q3.P$3; no longer D3.P$POS, U$5.P$3
- net N$24: now also D4.P$2, Q4.P$3; no longer D4.P$POS, U$6.P$3
- net N$25: now also U$7.SETC_XM; no longer U$7.P$8
- net N$26: now also U$7.SETP_XM; no longer U$7.P$9
- net N$27: now also U$7.C1_XM; no longer U$7.P$7
- net N$29: now also U$7.CS_G; no longer U$7.P$19
- net N$30: now also U$7.CS_XM; no longer U$7.P$20
- net PB5: now also Q1.P$1; no longer U$3.P$1
- net PE3: now also Q3.P$1; no longer U$5.P$1
- net PE4: now also Q4.P$1; no longer U$6.P$1
- net PE5: now also Q2.P$1; no longer U$4.P$1
- net SCK: now also J1.3
- net SCL: now also U$7.SCL; no longer U$7.P$21
- net SDA: now also U$7.SDA; no longer U$7.P$24
Other:
- note added: "1"
- note added: "1 of 1"
- note added: "ATMEGA128RFA1 Microcontroller"
- note added: "Daniel Knapp -- James Lee"
- note added: "In-System Programmer"
- note added: "Inertial Measurement Unit"
- note added: "Motor Drivers"
- note added: "Power Regulation"
- note added: "RF Antennae"
- note added: "Serial Debugger"
- note added: "Serial Programmer"
- moved on the sheet: B1, C1, C10, C11, C12, C13, C14, C15, C16, C17, C2, C3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

Commit message: Corrected Schematic and some of the board
Parts:
- C16, C17: device lab5_comps:C-USC0805 -> lab5_comps:R-US_R0805
Connections:
- removed net N$1: C14.2, S1.O, U$2.EN, U$2.IN
- new net VBAT: C14.2, D1.P$1, D2.P$1, D3.P$1, D4.P$1, MOT1.2, MOT2.2, MOT3.2, MOT4.2, S1.O, U$2.EN, U$2.IN
- net 3V: no longer D1.P$1, D2.P$1, D3.P$1, D4.P$1, MOT1.2, MOT2.2, MOT3.2, MOT4.2
Changed lines of the file:
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@@
 <setting verticaltext="up"/>
 </settings>
-<grid distance="0.05" unitdist="inch" unit="inch" style="lines" multiple="1" display="yes" altdistance="0.01" altunitdist="inch" altunit="inch"/>
+<grid distance="0.1" unitdist="inch" unit="inch" style="lines" multiple="1" display="no" altdistance="0.01" altunitdist="inch" altunit="inch"/>
 <layers>
 <layer number="1" name="Top" color="4" fill="1" visible="no" active="no"/>
@@
 <part name="C12" library="lab5_comps" deviceset="C-US" device="C0805" value="0.01uF"/>
 <part name="C14" library="lab5_comps" deviceset="C-US" device="C0805" value="1uF"/>
-<part name="C16" library="lab5_comps" deviceset="C-US" device="C0805" value="JUMP"/>
-<part name="C17" library="lab5_comps" deviceset="C-US" device="C0805" value="JUMP"/>
+<part name="C16" library="lab5_comps" deviceset="R-US_" device="R0805" value="JUMP"/>
+<part name="C17" library="lab5_comps" deviceset="R-US_" device="R0805" value="JUMP"/>
 <part name="J1" library="lab5_comps" deviceset="AVR_SPI_PRG_6" device="NS" value="ISP"/>
 <part name="JP1" library="lab5_comps" deviceset="FTDI_BASIC" device="PTH" value="FTDI"/>
@@
 <instance part="C12" gate="G$1" x="-119.38" y="76.2"/>
 <instance part="C14" gate="G$1" x="-157.48" y="93.98"/>
-<instance part="C16" gate="G$1" x="157.48" y="-68.58" rot="R90"/>
-<instance part="C17" gate="G$1" x="157.48" y="-88.9" rot="R90"/>
+<instance part="C16" gate="G$1" x="157.48" y="-68.58"/>
+<instance part="C17" gate="G$1" x="157.48" y="-88.9"/>
 <instance part="J1" gate="G$1" x="-53.34" y="86.36"/>
 <instance part="JP1" gate="G$1" x="-12.7" y="86.36" rot="MR180"/>
@@
 </segment>
 </net>
-<net name="N$1" class="0">
+<net name="VBAT" class="0">
 <segment>
 <pinref part="S1" gate="1" pin="O"/>
@@
 <wire x1="-149.86" y1="78.74" x2="-157.48" y2="78.74" width="0.1524" layer="91"/>
 <wire x1="-157.48" y1="78.74" x2="-157.48" y2="88.9" width="0.1524" layer="91"/>
+<label x="-157.48" y="78.74" size="1.016" layer="125" rot="R180" xref="yes"/>
+</segment>
+<segment>
+<wire x1="83.82" y1="96.52" x2="83.82" y2="88.9" width="0.1524" layer="91"/>
+<pinref part="MOT1" gate="G$1" pin="2"/>
+<wire x1="81.28" y1="88.9" x2="83.82" y2="88.9" width="0.1524" layer="91"/>
+<wire x1="83.82" y1="88.9" x2="91.44" y2="88.9" width="0.1524" layer="91"/>
+<wire x1="91.44" y1="88.9" x2="91.44" y2="86.36" width="0.1524" layer="91"/>
+<junction x="83.82" y="88.9"/>
+<label x="83.82" y="96.52" size="1.016" layer="95" rot="R90" xref="yes"/>
+<pinref part="D1" gate="G$1" pin="P$1"/>
+</segment>
+<segment>
+<wire x1="124.46" y1="96.52" x2="124.46" y2="88.9" width="0.1524" layer="91"/>
+<pinref part="MOT2" gate="G$1" pin="2"/>
+<wire x1="121.92" y1="88.9" x2="124.46" y2="88.9" width="0.1524" layer="91"/>
+<wire x1="124.46" y1="88.9" x2="132.08" y2="88.9" width="0.1524" layer="91"/>
+<wire x1="132.08" y1="88.9" x2="132.08" y2="86.36" width="0.1524" layer="91"/>
+<junction x="124.46" y="88.9"/>
+<label x="124.46" y="96.52" size="1.016" layer="95" rot="R90" xref="yes"/>
+<pinref part="D2" gate="G$1" pin="P$1"/>
+</segment>
+<segment>
+<wire x1="167.64" y1="96.52" x2="167.64" y2="88.9" width="0.1524" layer="91"/>
+<pinref part="MOT3" gate="G$1" pin="2"/>
+<wire x1="165.1" y1="88.9" x2="167.64" y2="88.9" width="0.1524" layer="91"/>
+<wire x1="167.64" y1="88.9" x2="175.26" y2="88.9" width="0.1524" layer="91"/>
+<wire x1="175.26" y1="88.9" x2="175.26" y2="86.36" width="0.1524" layer="91"/>
+<junction x="167.64" y="88.9"/>
+<label x="167.64" y="96.52" size="1.016" layer="95" rot="R90" xref="yes"/>
+<pinref part="D3" gate="G$1" pin="P$1"/>
+</segment>
+<segment>
+<wire x1="213.36" y1="96.52" x2="213.36" y2="88.9" width="0.1524" layer="91"/>
+<pinref part="MOT4" gate="G$1" pin="2"/>
+<wire x1="210.82" y1="88.9" x2="213.36" y2="88.9" width="0.1524" layer="91"/>
+<wire x1="213.36" y1="88.9" x2="220.98" y2="88.9" width="0.1524" layer="91"/>
+<wire x1="220.98" y1="88.9" x2="220.98" y2="86.36" width="0.1524" layer="91"/>
+<junction x="213.36" y="88.9"/>
+<label x="213.36" y="96.52" size="1.016" layer="95" rot="R90" xref="yes"/>
+<pinref part="D4" gate="G$1" pin="P$1"/>
 </segment>
 </net>
@@
 <wire x1="-99.06" y1="88.9" x2="-93.98" y2="88.9" width="0.1524" layer="91"/>
 <junction x="-99.06" y="88.9"/>
-<label x="-93.98" y="88.9" size="1.778" layer="95" xref="yes"/>
+<label x="-93.98" y="88.9" size="1.016" layer="95" xref="yes"/>
 </segment>
 <segment>
@@
 <wire x1="-45.72" y1="12.7" x2="-45.72" y2="15.24" width="0.1524" layer="91"/>
 <label x="-45.72" y="15.24" size="1.016" layer="95" rot="R90" xref="yes"/>
-</segment>
-<segment>
-<wire x1="83.82" y1="96.52" x2="83.82" y2="88.9" width="0.1524" layer="91"/>
-<pinref part="MOT1" gate="G$1" pin="2"/>
-<wire x1="81.28" y1="88.9" x2="83.82" y2="88.9" width="0.1524" layer="91"/>
-<wire x1="83.82" y1="88.9" x2="91.44" y2="88.9" width="0.1524" layer="91"/>
-<wire x1="91.44" y1="88.9" x2="91.44" y2="86.36" width="0.1524" layer="91"/>
-<junction x="83.82" y="88.9"/>
-<label x="83.82" y="96.52" size="1.016" layer="95" rot="R90" xref="yes"/>
-<pinref part="D1" gate="G$1" pin="P$1"/>
-</segment>
-<segment>
-<wire x1="124.46" y1="96.52" x2="124.46" y2="88.9" width="0.1524" layer="91"/>
-<pinref part="MOT2" gate="G$1" pin="2"/>
-<wire x1="121.92" y1="88.9" x2="124.46" y2="88.9" width="0.1524" layer="91"/>
-<wire x1="124.46" y1="88.9" x2="132.08" y2="88.9" width="0.1524" layer="91"/>
-<wire x1="132.08" y1="88.9" x2="132.08" y2="86.36" width="0.1524" layer="91"/>
-<junction x="124.46" y="88.9"/>
-<label x="124.46" y="96.52" size="1.016" layer="95" rot="R90" xref="yes"/>
-<pinref part="D2" gate="G$1" pin="P$1"/>
-</segment>
-<segment>
-<wire x1="167.64" y1="96.52" x2="167.64" y2="88.9" width="0.1524" layer="91"/>
-<pinref part="MOT3" gate="G$1" pin="2"/>
-<wire x1="165.1" y1="88.9" x2="167.64" y2="88.9" width="0.1524" layer="91"/>
-<wire x1="167.64" y1="88.9" x2="175.26" y2="88.9" width="0.1524" layer="91"/>
-<wire x1="175.26" y1="88.9" x2="175.26" y2="86.36" width="0.1524" layer="91"/>
-<junction x="167.64" y="88.9"/>
-<label x="167.64" y="96.52" size="1.016" layer="95" rot="R90" xref="yes"/>
-<pinref part="D3" gate="G$1" pin="P$1"/>
-</segment>
-<segment>
-<wire x1="213.36" y1="96.52" x2="213.36" y2="88.9" width="0.1524" layer="91"/>
-<pinref part="MOT4" gate="G$1" pin="2"/>
-<wire x1="210.82" y1="88.9" x2="213.36" y2="88.9" width="0.1524" layer="91"/>
-<wire x1="213.36" y1="88.9" x2="220.98" y2="88.9" width="0.1524" layer="91"/>
-<wire x1="220.98" y1="88.9" x2="220.98" y2="86.36" width="0.1524" layer="91"/>
-<junction x="213.36" y="88.9"/>
-<label x="213.36" y="96.52" size="1.016" layer="95" rot="R90" xref="yes"/>
-<pinref part="D4" gate="G$1" pin="P$1"/>
 </segment>
 <segment>
@@
 <segment>
 <pinref part="C16" gate="G$1" pin="1"/>
-<wire x1="154.94" y1="-68.58" x2="142.24" y2="-68.58" width="0.1524" layer="91"/>
+<wire x1="152.4" y1="-68.58" x2="142.24" y2="-68.58" width="0.1524" layer="91"/>
 <wire x1="142.24" y1="-68.58" x2="142.24" y2="-83.82" width="0.1524" layer="91"/>
 <label x="142.24" y="-83.82" size="1.016" layer="95" rot="R180" xref="yes"/>
@@
 <wire x1="142.24" y1="-86.36" x2="142.24" y2="-88.9" width="0.1524" layer="91"/>
 <pinref part="C17" gate="G$1" pin="1"/>
-<wire x1="142.24" y1="-88.9" x2="154.94" y2="-88.9" width="0.1524" layer="91"/>
+<wire x1="142.24" y1="-88.9" x2="152.4" y2="-88.9" width="0.1524" layer="91"/>
 <label x="142.24" y="-86.36" size="1.016" layer="95" rot="R180" xref="yes"/>
 </segment>

Commit message: finisehd board. but need to add names
Connections:
- net GND: no longer U1.PADDLE
- net PB5: now also Q2.P$1, R6.2; no longer Q1.P$1, R5.2
- net PE5: now also Q1.P$1, R5.2; no longer Q2.P$1, R6.2
