File: Lab6/lab6.sch (EAGLE design)
At the start: 54 parts, among them J1 ISP, Q1 SI2302CDS, Q2 SI2302CDS, Q3 SI2302CDS, Q4 SI2302CDS, U1 ATMEGA128RFA1, Y1 16MHz

Commit message: Fixed What Swanson Wanted
Connections:
- net RFN renamed RF_N
- net RFP renamed RF_P
Changed lines of the file:
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@@
 </segment>
 </net>
-<net name="RFP" class="0">
+<net name="RF_P" class="0">
 <segment>
 <wire x1="-17.78" y1="-33.02" x2="-15.24" y2="-33.02" width="0.1524" layer="91"/>
@@
 </segment>
 </net>
-<net name="RFN" class="0">
+<net name="RF_N" class="0">
 <segment>
 <wire x1="-17.78" y1="-35.56" x2="-15.24" y2="-35.56" width="0.1524" layer="91"/>
